File: hardware/hardware.kicad_sch (KiCad schematic)
At the start: 59 parts, among them J1 SMA, J2 Test Header, P5 BMIS-202-C, U1 CC1101, U2 CC1190, U3 B39921B3588U410, X1 26.000 MHz

Commit message: Worked on footprints and hardware definations.
Parts:
- C1, C30: footprint Capacitor_SMD:C_0402_1005Metric -> Capacitor_SMD:C_0603_1608Metric; Digikey Link (none) -> https://www.digikey.com/en/products/detail/murata-electroni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; Digikey Part Number (none) -> 490-GRM188R61C105KA12JCT-ND
- C101, C132: footprint Capacitor_SMD:C_0402_1005Metric -> Capacitor_SMD:C_0603_1608Metric; Digikey Link (none) -> https://www.digikey.com/en/products/detail/kemet/CBR06C150J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; Digikey Part Number (none) -> 399-CBR06C150J5GACAUTOCT-ND
- C111, C141, C151, C181, C41, C51, C91: footprint Capacitor_SMD:C_0402_1005Metric -> Capacitor_SMD:C_0805_2012Metric; Digikey Link (none) -> https://www.digikey.com/en/products/detail/kyocera-avx/KGM2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; Digikey Part Number (none) -> 478-KGM21NR71H104KTCT-ND
- C121: footprint Capacitor_SMD:C_0402_1005Metric -> Capacitor_SMD:C_0603_1608Metric; Digikey Link (none) -> https://www.digikey.com/en/products/detail/kemet/CBR06C199B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; Digikey Part Number (none) -> 399-16151-1-ND - Cut Tape (CT
- C122, C131: footprint Capacitor_SMD:C_0402_1005Metric -> Capacitor_SMD:C_0805_2012Metric; Digikey Link (none) -> https://www.digikey.com/en/products/detail/murata-electroni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; Digikey Part Number (none) -> 490-5282-1-ND - Cut Tape (CT)
- C123, C21, C26: footprint Capacitor_SMD:C_0402_1005Metric -> Capacitor_SMD:C_0603_1608Metric; Digikey Link (none) -> https://www.digikey.com/en/products/detail/kemet/CBR06C470J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; Digikey Part Number (none) -> 399-17536-1-ND
- C124: footprint Capacitor_SMD:C_0402_1005Metric -> Capacitor_SMD:C_0805_2012Metric; Digikey Link (none) -> https://www.digikey.com/en/products/detail/kyocera-avx/KGQ2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; Digikey Part Number (none) -> 478-KGQ21HCG2D101JTCT-ND
- C125: footprint Capacitor_SMD:C_0402_1005Metric -> Capacitor_SMD:C_0805_2012Metric; Digikey Link (none) -> https://www.digikey.com/en/products/detail/murata-electroni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; Digikey Part Number (none) -> 490-GQM2195G2ER80BB12DCT-ND - Cut Tape (CT)
- C161: footprint Capacitor_SMD:C_0402_1005Metric -> Capacitor_SMD:C_0805_2012Metric; Digikey Link (none) -> https://www.digikey.com/en/products/detail/kyocera-avx/0805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; Digikey Part Number (none) -> 478-KGQ21HCG2D270JTCT-ND
- C2: footprint Capacitor_SMD:C_0402_1005Metric -> Capacitor_SMD:C_0603_1608Metric; Digikey Link (none) -> https://www.digikey.com/en/products/detail/murata-electroni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; Digikey Part Number (none) -> 490-12538-1-ND
- C22, C52, C81: footprint Capacitor_SMD:C_0402_1005Metric -> Capacitor_SMD:C_0603_1608Metric; Digikey Link (none) -> https://www.digikey.com/en/products/detail/kemet/CBR06C120J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; Digikey Part Number (none) -> 399-CBR06C120J5GACCT-ND
- C24: footprint Capacitor_SMD:C_0402_1005Metric -> Capacitor_SMD:C_0805_2012Metric; Digikey Link (none) -> https://www.digikey.com/en/products/detail/murata-electroni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; Digikey Part Number (none) -> 490-GQM2195C2E3R3CB12DCT-ND - Cut Tape (CT)
- C25: footprint Capacitor_SMD:C_0402_1005Metric -> Capacitor_SMD:C_1206_3216Metric; Digikey Link (none) -> https://www.digikey.com/en/products/detail/kemet/CBR06C759B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; Digikey Part Number (none) -> 399-16247-1-ND - Cut Tape (CT)
- C27: footprint Capacitor_SMD:C_0402_1005Metric -> Capacitor_SMD:C_0805_2012Metric; Digikey Link (none) -> https://www.digikey.com/en/products/detail/vishay-vitramon/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; Digikey Part Number (none) -> 720-VJ0805D102JXJQJHTCT-ND
- C28: footprint Capacitor_SMD:C_0402_1005Metric -> Capacitor_SMD:C_1206_3216Metric; now not fitted
- C3: footprint Capacitor_SMD:C_0402_1005Metric -> Capacitor_SMD:C_0603_1608Metric; Digikey Link (none) -> https://www.digikey.com/en/products/detail/vishay-vitramon/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; Digikey Part Number (none) -> 720-VJ0603D221JXJQJHTCT-ND
- FB1: footprint (none) -> Inductor_SMD:L_1206_3216Metric
- J1: footprint (none) -> Connector_Coaxial:SMA_Molex_73251-1153_EdgeMount_Horizontal
- J2: footprint Connector_PinSocket_2.54mm:PinSocket_2x12_P2.54mm_Vertical -> Connector_PinHeader_2.54mm:PinHeader_2x12_P2.54mm_Vertical
- L121, L131: footprint (none) -> Inductor_SMD:L_0603_1608Metric; Digikey Link (none) -> https://www.digikey.com/en/products/detail/murata-electroni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; Digikey Part Number (none) -> 490-15799-1-ND
- L122, L132: footprint (none) -> Inductor_SMD:L_0603_1608Metric; Digikey Link (none) -> https://www.digikey.com/en/products/detail/murata-electroni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; Digikey Part Number (none) -> 490-15805-1-ND
- L130: footprint (none) -> Inductor_SMD:L_1206_3216Metric; Digikey Link (none) -> https://www.digikey.com/en/products/detail/murata-electroni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; Digikey Part Number (none) -> 490-1100-1-ND
- L2: footprint (none) -> Inductor_SMD:L_0603_1608Metric; Digikey Link (none) -> https://www.digikey.com/en/products/detail/murata-electroni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; Digikey Part Number (none) -> 490-LQW18AS11NG00DCT-ND
- L21: footprint (none) -> Inductor_SMD:L_0603_1608Metric; Digikey Link (none) -> https://www.digikey.com/en/products/detail/murata-electroni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; Digikey Part Number (none) -> 490-LQW18AS22NG00DCT-ND
- L22: footprint (none) -> Inductor_SMD:L_0603_1608Metric; Digikey Link (none) -> https://www.digikey.com/en/products/detail/murata-electroni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; Digikey Part Number (none) -> 490-LQW18AS7N5G00DCT-ND
- L23: footprint (none) -> Inductor_SMD:L_0402_1005Metric; Digikey Link (none) -> https://www.digikey.com/en/products/detail/murata-electroni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; Digikey Part Number (none) -> 490-LQG15WZ2N9B02DCT-ND
- L24: footprint (none) -> Inductor_SMD:L_0402_1005Metric; Digikey Link (none) -> https://www.digikey.com/en/products/detail/murata-electroni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; Digikey Part Number (none) -> 490-LQG15HS9N1G02DCT-ND
- L25: footprint (none) -> Inductor_SMD:L_0603_1608Metric; Digikey Link (none) -> https://www.digikey.com/en/products/detail/murata-electroni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; Digikey Part Number (none) -> 490-LQW18AS10NG00DCT-ND
- P5: footprint (none) -> RF_Shielding:Laird_Technologies_BMI-S-202-F_16.50x16.50mm
- R141: footprint (none) -> Resistor_SMD:R_1206_3216Metric
- R151, R161, R171: footprint Resistor_SMD:R_0402_1005Metric -> Resistor_SMD:R_1206_3216Metric
- TP1, TP2: footprint (none) -> Connector_PinHeader_2.54mm:PinHeader_1x01_P2.54mm_Vertical
- X1: footprint (none) -> Crystal:Crystal_SMD_3225-4Pin_3.2x2.5mm
