File: hardware/I2C0.kicad_sch (KiCad schematic)
At the start: 15 parts, among them U4 ADS1115IDGS, U5 BME280

Commit message: More work on the scehmatic for I2C0 and I2C1 + UART GPS.
Parts:
- removed JP1: SolderJumper_2_Open, symbol Jumper:SolderJumper_2_Open
- removed R01, R02, R03, R06, R09: 10K, symbol Device:R_US
- R07, R08: value 10K -> 4.7 K
Connections:
- net GNDREF: now also U4.1 (ADDR), U5.5 (SDO)
- net I2C0_SCL: now also R08.2, U4.10 (SCL), U5.4 (SCK)
- net I2C0_SDA: now also R07.2, U4.9 (SDA), U5.3 (SDI)
- net VDD: now also R07.1, R08.1, U5.2 (CSB)

Commit message: Finished rough draft of the schematic.
Connections:
- net GNDREF renamed GND
Changed lines of the file:
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@@
 			)
 		)
-		(property "Value" "GNDREF"
-			(at 105.41 101.6 0)
-			(show_name no)
-			(do_not_autoplace no)
-			(effects
-				(font
-					(size 1.27 1.27)
-				)
+		(property "Value" "GND"
+			(at 107.95 97.7899 0)
+			(show_name no)
+			(do_not_autoplace no)
+			(effects
+				(font
+					(size 1.27 1.27)
+				)
+				(justify left)
 			)
 		)
@@
 			)
 		)
-		(property "Value" "GNDREF"
-			(at 95.25 146.05 0)
-			(show_name no)
-			(do_not_autoplace no)
-			(effects
-				(font
-					(size 1.27 1.27)
-				)
+		(property "Value" "GND"
+			(at 97.79 142.2399 0)
+			(show_name no)
+			(do_not_autoplace no)
+			(effects
+				(font
+					(size 1.27 1.27)
+				)
+				(justify left)
 			)
 		)
@@
 			)
 		)
-		(property "Value" "GNDREF"
-			(at 88.9 102.87 0)
-			(show_name no)
-			(do_not_autoplace no)
-			(effects
-				(font
-					(size 1.27 1.27)
-				)
+		(property "Value" "GND"
+			(at 91.44 99.0599 0)
+			(show_name no)
+			(do_not_autoplace no)
+			(effects
+				(font
+					(size 1.27 1.27)
+				)
+				(justify left)
 			)
 		)
@@
 			)
 		)
-		(property "Value" "GNDREF"
-			(at 160.02 111.76 0)
-			(show_name no)
-			(do_not_autoplace no)
-			(effects
-				(font
-					(size 1.27 1.27)
-				)
+		(property "Value" "GND"
+			(at 162.56 107.9499 0)
+			(show_name no)
+			(do_not_autoplace no)
+			(effects
+				(font
+					(size 1.27 1.27)
+				)
+				(justify left)
 			)
 		)
@@
 			)
 		)
-		(property "Value" "GNDREF"
-			(at 55.88 111.76 0)
-			(show_name no)
-			(do_not_autoplace no)
-			(effects
-				(font
-					(size 1.27 1.27)
-				)
+		(property "Value" "GND"
+			(at 58.42 107.9499 0)
+			(show_name no)
+			(do_not_autoplace no)
+			(effects
+				(font
+					(size 1.27 1.27)
+				)
+				(justify left)
 			)
 		)
@@
 			)
 		)
-		(property "Value" "GNDREF"
-			(at 200.66 111.76 0)
-			(show_name no)
-			(do_not_autoplace no)
-			(effects
-				(font
-					(size 1.27 1.27)
-				)
-			)
-		)
+		(property "Value" "GND"
+			(at 203.2 107.9499 0)
+			(show_name no)
+			(do_not_autoplace no)
+			(effects
+				(font
+					(size 1.27 1.27)
+				)
+				(justify left)
+			)
+		)

Commit message: Fixed EEC errors.
Parts:
- R05: value 10K -> 10K OHM 0.1% 0.4W AXIAL; footprint (none) -> Resistor_THT:R_Axial_DIN0207_L6.3mm_D2.5mm_P7.62mm_Horizontal
- RT1: footprint (none) -> footprints:PPG102JA
Connections:
- no-connect marks 0 -> 2
Changed lines of the file:
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@@
 		(color 0 0 0 0)
+	)
+	(no_connect
+		(at 73.66 106.68)
+	)
+	(no_connect
+		(at 81.28 106.68)
 	)
 	(wire
@@
 			)
 		)
-		(property "Footprint" ""
+		(property "Footprint" "footprints:PPG102JA"
 			(at 59.69 139.7 0)
 			(hide yes)
@@
 			)
 		)
-		(property "Value" "10K"
-			(at 67.056 127 0)
+		(property "Value" "10K OHM 0.1% 0.4W AXIAL"
+			(at 45.974 126.746 0)
 			(show_name no)
 			(do_not_autoplace no)
@@
 			)
 		)
-		(property "Footprint" ""
+		(property "Footprint" "Resistor_THT:R_Axial_DIN0207_L6.3mm_D2.5mm_P7.62mm_Horizontal"
 			(at 74.676 125.984 90)
 			(hide yes)
@@
 			)
 		)
-		(property "Datasheet" ""
+		(property "Datasheet" "kicad-embed://mbsmapre.pdf"
 			(at 73.66 125.73 0)
 			(hide yes)
@@
 			)
 		)
-		(property "Description" "Resistor, US symbol"
+		(property "Description" "10 kOhms ±0.1% 0.4W Through Hole Resistor Axial Metal Film"
 			(at 73.66 125.73 0)
 			(hide yes)

Commit message: Added footprints for the resitors.
Parts:
- R04, R07, R08: footprint (none) -> Resistor_SMD:R_1206_3216Metric
Changed lines of the file:
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@@
 			)
 		)
-		(property "Footprint" ""
+		(property "Footprint" "Resistor_SMD:R_1206_3216Metric"
 			(at 239.776 84.074 90)
 			(hide yes)
@@
 			)
 		)
-		(property "Footprint" ""
+		(property "Footprint" "Resistor_SMD:R_1206_3216Metric"
 			(at 249.936 84.074 90)
 			(hide yes)
@@
 			)
 		)
-		(property "Footprint" ""
+		(property "Footprint" "Resistor_SMD:R_1206_3216Metric"
 			(at 83.566 76.454 90)
 			(hide yes)

Commit message: Added capacitor footprints.
Parts:
- C01, C02: footprint (none) -> Capacitor_SMD:C_1206_3216Metric
Changed lines of the file:
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@@
 			)
 		)
-		(property "Footprint" ""
+		(property "Footprint" "Capacitor_SMD:C_1206_3216Metric"
 			(at 160.9852 106.68 0)
 			(hide yes)
@@
 			)
 		)
-		(property "Footprint" ""
+		(property "Footprint" "Capacitor_SMD:C_1206_3216Metric"
 			(at 56.8452 106.68 0)
 			(hide yes)

Commit message: Worked on footprints and hardware definations.
Parts:
- C01, C02: footprint Capacitor_SMD:C_1206_3216Metric -> Capacitor_SMD:C_0603_1608Metric; Digikey Link (none) -> https://www.digikey.com/en/products/detail/murata-electroni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; Digikey Part Number (none) -> 490-12538-1-ND
- R07, R08: value 4.7 K -> 4.7k
Connections:
- net GND: now also U4.7 (AIN3); no longer U4.6 (AIN2)
Changed lines of the file:
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@@
 	)
 	(no_connect
-		(at 81.28 106.68)
+		(at 78.74 106.68)
 	)
 	(wire
@@
 	(wire
 		(pts
-			(xy 78.74 109.22) (xy 78.74 106.68)
-		)
-		(stroke
-			(width 0)
-			(type default)
-		)
-	)
-	(wire
-		(pts
 			(xy 200.66 93.98) (xy 200.66 99.06)
 		)
@@
 	(wire
 		(pts
+			(xy 81.28 109.22) (xy 86.36 109.22)
+		)
+		(stroke
+			(width 0)
+			(type default)
+		)
+	)
+	(wire
+		(pts
 			(xy 163.83 96.52) (xy 160.02 96.52)
 		)
@@
 	(wire
 		(pts
+			(xy 81.28 106.68) (xy 81.28 109.22)
+		)
+		(stroke
+			(width 0)
+			(type default)
+		)
+	)
+	(wire
+		(pts
 			(xy 48.26 96.52) (xy 55.88 96.52)
-		)
-		(stroke
-			(width 0)
-			(type default)
-		)
-	)
-	(wire
-		(pts
-			(xy 86.36 109.22) (xy 78.74 109.22)
 		)
 		(stroke
@@
 			)
 		)
-		(property "Value" "4.7 K"
+		(property "Value" "4.7k"
 			(at 241.3 85.0899 0)
 			(show_name no)
@@
 			)
 		)
-		(property "Footprint" "Capacitor_SMD:C_1206_3216Metric"
+		(property "Footprint" "Capacitor_SMD:C_0603_1608Metric"
 			(at 160.9852 106.68 0)
 			(hide yes)
@@
 		)
 		(property "Description" "Unpolarized capacitor"
+			(at 160.02 102.87 0)
+			(hide yes)
+			(show_name no)
+			(do_not_autoplace no)
+			(effects
+				(font
+					(size 1.27 1.27)
+				)
+			)
+		)
+		(property "Digikey Link" "https://www.digikey.com/en/products/detail/murata-electronics/GRM188R60J106KE47D/5797506"
+			(at 160.02 102.87 0)
+			(hide yes)
+			(show_name no)
+			(do_not_autoplace no)
+			(effects
+				(font
+					(size 1.27 1.27)
+				)
+			)
+		)
+		(property "Digikey Part Number" "490-12538-1-ND"
 			(at 160.02 102.87 0)
 			(hide yes)
@@
 			)
 		)
-		(property "Value" "4.7 K"
+		(property "Value" "4.7k"
 			(at 251.46 85.0899 0)
 			(show_name no)
@@
 			)
 		)
-		(property "Footprint" "Capacitor_SMD:C_1206_3216Metric"
+		(property "Footprint" "Capacitor_SMD:C_0603_1608Metric"
 			(at 56.8452 106.68 0)
 			(hide yes)
@@
 			(at 55.88 102.87 0)
 			(hide yes)
+			(show_name no)
+			(do_not_autoplace no)
+			(effects
+				(font
+					(size 1.27 1.27)
+				)
+			)
+		)
+		(property "Digikey Link" "https://www.digikey.com/en/products/detail/murata-electronics/GRM188R60J106KE47D/5797506"
+			(at 55.88 102.87 0)
+			(hide yes)
+			(show_name no)
+			(do_not_autoplace no)
+			(effects
+				(font
+					(size 1.27 1.27)
+				)
+			)
+		)
+		(property "Digikey Part Number" "490-12538-1-ND"
+			(at 55.88 102.87 0)
+			(hide yes)

Commit message: Worked on PCB routing and component placement.
Parts:
- R04: footprint Resistor_SMD:R_1206_3216Metric -> Resistor_SMD:R_0603_1608Metric; Digikey Link (none) -> https://www.digikey.com/en/products/detail/vishay/MCT06030C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; Digikey Part Number (none) -> MCT0603-10.0K-CFCT-ND
- R05: Digikey Link (none) -> https://www.digikey.com/en/products/detail/vishay-beyschlag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; Digikey Part Number (none) -> BC4515CT-ND
- R07, R08: footprint Resistor_SMD:R_1206_3216Metric -> Resistor_SMD:R_0603_1608Metric; Digikey Link (none) -> https://www.digikey.com/en/products/detail/vishay/MCT06030C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; Digikey Part Number (none) -> MCT0603-4.70K-CFCT-ND
- RT1: Digikey Link (none) -> https://www.digikey.com/en/products/detail/littelfuse-ibu/P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; Digikey Part Number (none) -> 5666-PPG102JA-ND
- U4: Digikey Link (none) -> https://www.digikey.com/en/products/detail/texas-instrument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; Digikey Part Number (none) -> 296-38849-1-ND
- U5: Digikey Link (none) -> https://www.digikey.com/en/products/detail/bosch-sensortec/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; Digikey Part Number (none) -> 828-1063-1-ND
Changed lines of the file:
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@@
+			)
+		)
+		(property "Digikey Link" "https://www.digikey.com/en/products/detail/littelfuse-ibu/PPG102JA/10500302?s=N4IgTCBcDaIA5wOYEYAMYBWBDEBdAvkA"
+			(at 59.69 139.7 0)
+			(hide yes)
+			(show_name no)
+			(do_not_autoplace no)
+			(effects
+				(font
+					(size 1.27 1.27)
+				)
+			)
+		)
+		(property "Digikey Part Number" "5666-PPG102JA-ND"
+			(at 59.69 139.7 0)
+			(hide yes)
+			(show_name no)
+			(do_not_autoplace no)
+			(effects
+				(font
+					(size 1.27 1.27)
+				)
 			)
 		)
@@
 			)
 		)
-		(property "Footprint" "Resistor_SMD:R_1206_3216Metric"
+		(property "Footprint" "Resistor_SMD:R_0603_1608Metric"
 			(at 239.776 84.074 90)
 			(hide yes)
@@
 		)
 		(property "Description" "Resistor, US symbol"
+			(at 238.76 83.82 0)
+			(hide yes)
+			(show_name no)
+			(do_not_autoplace no)
+			(effects
+				(font
+					(size 1.27 1.27)
+				)
+			)
+		)
+		(property "Digikey Link" "https://www.digikey.com/en/products/detail/vishay/MCT06030C4701FP500/2607853"
+			(at 238.76 83.82 0)
+			(hide yes)
+			(show_name no)
+			(do_not_autoplace no)
+			(effects
+				(font
+					(size 1.27 1.27)
+				)
+			)
+		)
+		(property "Digikey Part Number" "MCT0603-4.70K-CFCT-ND"
 			(at 238.76 83.82 0)
 			(hide yes)
@@
 			)
 		)
+		(property "Digikey Link" "https://www.digikey.com/en/products/detail/vishay-beyschlag-draloric-bc-components/MBB0207VE1002BC100/7350421?s=N4IgTCBcDaIEYGMAsBWAjChAXAtAOwBMQBdAXyA"
+			(at 73.66 125.73 0)
+			(hide yes)
+			(show_name no)
+			(do_not_autoplace no)
+			(effects
+				(font
+					(size 1.27 1.27)
+				)
+			)
+		)
+		(property "Digikey Part Number" "BC4515CT-ND"
+			(at 73.66 125.73 0)
+			(hide yes)
+			(show_name no)
+			(do_not_autoplace no)
+			(effects
+				(font
+					(size 1.27 1.27)
+				)
+			)
+		)
 		(pin "2"
 		)
@@
 			)
 		)
-		(property "Footprint" "Resistor_SMD:R_1206_3216Metric"
+		(property "Footprint" "Resistor_SMD:R_0603_1608Metric"
 			(at 249.936 84.074 90)
 			(hide yes)
@@
 		)
 		(property "Description" "Resistor, US symbol"
+			(at 248.92 83.82 0)
+			(hide yes)
+			(show_name no)
+			(do_not_autoplace no)
+			(effects
+				(font
+					(size 1.27 1.27)
+				)
+			)
+		)
+		(property "Digikey Link" "https://www.digikey.com/en/products/detail/vishay/MCT06030C4701FP500/2607853"
+			(at 248.92 83.82 0)
+			(hide yes)
+			(show_name no)
+			(do_not_autoplace no)
+			(effects
+				(font
+					(size 1.27 1.27)
+				)
+			)
+		)
+		(property "Digikey Part Number" "MCT0603-4.70K-CFCT-ND"
 			(at 248.92 83.82 0)
 			(hide yes)
@@
 			)
 		)
+		(property "Digikey Link" "https://www.digikey.com/en/products/detail/bosch-sensortec/BME280/6136306"
+			(at 182.88 96.52 90)
+			(hide yes)
+			(show_name no)
+			(do_not_autoplace no)
+			(effects
+				(font
+					(size 1.27 1.27)
+				)
+			)
+		)
+		(property "Digikey Part Number" "828-1063-1-ND"
+			(at 182.88 96.52 90)
+			(hide yes)
+			(show_name no)
+			(do_not_autoplace no)
+			(effects
+				(font
+					(size 1.27 1.27)
+				)
+			)
+		)
 		(pin "4"
 		)
@@
 			)
 		)
-		(property "Footprint" "Resistor_SMD:R_1206_3216Metric"
+		(property "Footprint" "Resistor_SMD:R_0603_1608Metric"
 			(at 83.566 76.454 90)
 			(hide yes)
@@
 		)
 		(property "Description" "Resistor, US symbol"
+			(at 82.55 76.2 0)
+			(hide yes)
+			(show_name no)
+			(do_not_autoplace no)
+			(effects
+				(font
+					(size 1.27 1.27)
+				)
+			)
+		)
+		(property "Digikey Link" "https://www.digikey.com/en/products/detail/vishay/MCT06030C1002FP500/1850440"
+			(at 82.55 76.2 0)
+			(hide yes)
+			(show_name no)
+			(do_not_autoplace no)
+			(effects
+				(font
+					(size 1.27 1.27)
+				)
+			)
+		)
+		(property "Digikey Part Number" "MCT0603-10.0K-CFCT-ND"
 			(at 82.55 76.2 0)
 			(hide yes)
@@
 			(hide yes)
 			(show_name no)
+			(do_not_autoplace no)
+			(effects
+				(font
+					(size 1.27 1.27)
+				)
+			)
+		)
+		(property "Digikey Link" "https://www.digikey.com/en/products/detail/texas-instruments/ADS1115IDGSR/2231567"
+			(at 76.2 96.52 90)
+			(hide yes)
+			(show_name no)
+			(do_not_autoplace no)
+			(effects
+				(font
+					(size 1.27 1.27)
+				)
+			)
+		)
+		(property "Digikey Part Number" "296-38849-1-ND"
+			(at 76.2 96.52 90)
+			(hide yes)
+			(show_name no)
