File: hardware/SDCard_VDD.kicad_sch (KiCad schematic)
At the start: 0 parts

Commit message: Finished rough draft of the schematic.
Parts:
- added B41: 1079, 1079_KEY, symbol 2026-07-24_00-32-24:1079
- added C44: 680 uF, symbol Device:C
- added C45: 330/35 uF/V, symbol Device:C
- added C46: 01. uF, symbol Device:C
- added D41: 1N5820, Diode_THT:D_DO-201AD_P15.24mm_Horizontal, symbol Diode:1N5820
- added J3: Micro_SD_Card, symbol Connector:Micro_SD_Card
- added L43: 33 uH, symbol Device:L
- added SW41: SW_DPST_x2, symbol Switch:SW_DPST_x2
- added U8: LM2596S-3.3, Package_TO_SOT_SMD:TO-263-5_TabPin3, symbol Regulator_Switching:LM2596S-3.3
Connections:
- new net: C44.1, SW41.2 (B), U8.1 (VIN)
- new net: D41.1 (K), L43.2, U8.2 (OUT)
- new net: B41.1, SW41.1 (A)
- new net: B41.2, B41.4
- new net GND: B41.3, C44.2, C45.2, C46.2, D41.2 (A), J3.6 (VSS), U8.3 (GND), U8.5 (~{ON}/OFF)
- new net SD_CSn: J3.2 (DAT3/CD)
- new net SD_RX: J3.7 (DAT0)
- new net SD_SCK: J3.5 (CLK)
- new net SD_TX: J3.3 (CMD)
- new net VDD: C45.1, C46.1, J3.4 (VDD), L43.1, U8.4 (FB)
- no-connect marks 0 -> 3
Other:
- note added: "This is set up for a SPI microsd connection"

Commit message: Fixed EEC errors.
Parts:
- removed J3: Micro_SD_Card, symbol Connector:Micro_SD_Card
- removed SW41: SW_DPST_x2, symbol Switch:SW_DPST_x2
- added J4: Micro_SD_Card_Det1, symbol Connector:Micro_SD_Card_Det1
- added SW41: SW_SPST, symbol Switch:SW_SPST
- B41: footprint 1079_KEY -> footprints:1079_KEY
- C44: value 680 uF -> 180 uF
- C46: value 01. uF -> 0.1 uF
Connections:
- net GND: now also J4.6 (VSS), J4.SH (SHIELD)
- net SD_CSn: now also J4.2 (DAT3/CD)
- net SD_RX: now also J4.7 (DAT0)
- net SD_SCK: now also J4.5 (CLK)
- net SD_TX: now also J4.3 (CMD)
- net VDD: now also J4.4 (VDD)
- net at C44.1, U8.1 (VIN): now also SW41.2 (B)
- net at B41.1: now also SW41.1 (A)
- new net SD_DETECT: J4.9 (DET)
- no-connect marks 3 -> 2
Changed lines of the file:
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@@
-	)
-	(no_connect
-		(at 166.37 143.51)
 	)
 	(no_connect
@@
 	(wire
 		(pts
+			(xy 106.68 143.51) (xy 123.19 143.51)
+		)
+		(stroke
+			(width 0)
+			(type default)
+		)
+	)
+	(wire
+		(pts
 			(xy 193.04 67.31) (xy 193.04 71.12)
 		)
@@
 	(wire
 		(pts
+			(xy 167.64 143.51) (xy 167.64 144.78)
+		)
+		(stroke
+			(width 0)
+			(type default)
+		)
+	)
+	(wire
+		(pts
 			(xy 63.5 57.15) (xy 63.5 63.5)
 		)
@@
 		(pts
 			(xy 154.94 71.12) (xy 154.94 67.31)
+		)
+		(stroke
+			(width 0)
+			(type default)
+		)
+	)
+	(wire
+		(pts
+			(xy 166.37 143.51) (xy 167.64 143.51)
 		)
 		(stroke
@@
 		(property "Intersheetrefs" "${INTERSHEET_REFS}"
 			(at 97.7682 135.89 0)
+			(hide yes)
+			(show_name no)
+			(do_not_autoplace no)
+			(effects
+				(font
+					(size 1.27 1.27)
+				)
+				(justify right)
+			)
+		)
+	)
+	(global_label "SD_DETECT"
+		(shape output)
+		(at 106.68 143.51 180)
+		(fields_autoplaced yes)
+		(effects
+			(font
+				(size 1.27 1.27)
+			)
+			(justify right)
+		)
+		(property "Intersheetrefs" "${INTERSHEET_REFS}"
+			(at 93.4745 143.51 0)
 			(hide yes)
 			(show_name no)
@@
 	)
 	(symbol
-		(lib_id "Connector:Micro_SD_Card")
-		(at 146.05 128.27 0)
-		(unit 1)
-		(body_style 1)
-		(exclude_from_sim no)
-		(in_bom yes)
-		(on_board yes)
-		(in_pos_files yes)
-		(dnp no)
-		(fields_autoplaced yes)
-		(property "Reference" "J3"
-			(at 146.685 109.22 0)
-			(show_name no)
-			(do_not_autoplace no)
-			(effects
-				(font
-					(size 1.27 1.27)
-				)
-			)
-		)
-		(property "Value" "Micro_SD_Card"
-			(at 146.685 111.76 0)
-			(show_name no)
-			(do_not_autoplace no)
-			(effects
-				(font
-					(size 1.27 1.27)
-				)
-			)
-		)
-		(property "Footprint" ""
-			(at 175.26 120.65 0)
-			(hide yes)
-			(show_name no)
-			(do_not_autoplace no)
-			(effects
-				(font
-					(size 1.27 1.27)
-				)
-			)
-		)
-		(property "Datasheet" "https://www.we-online.com/components/products/datasheet/693072010801.pdf"
-			(at 146.05 128.27 0)
-			(hide yes)
-			(show_name no)
-			(do_not_autoplace no)
-			(effects
-				(font
-					(size 1.27 1.27)
-				)
-			)
-		)
-		(property "Description" "Micro SD Card Socket"
-			(at 146.05 128.27 0)
-			(hide yes)
-			(show_name no)
-			(do_not_autoplace no)
-			(effects
-				(font
-					(size 1.27 1.27)
-				)
-			)
-		)
-		(pin "SH"
-		)
-		(pin "3"
-		)
-		(pin "1"
-		)
-		(pin "5"
-		)
-		(pin "6"
-		)
-		(pin "7"
-		)
-		(pin "8"
-		)
-		(pin "2"
-		)
-		(pin "4"
-		)
-		(instances
-			(project "hardware"
-				(path "/63c7c074-dbc9-4433-b26d-8a099c78afdf/43eeeb2a-883a-4738-8b2b-317d62bf6c96"
-					(reference "J3")
-					(unit 1)
-				)
-			)
-		)
-	)
-	(symbol
 		(lib_id "Regulator_Switching:LM2596S-3.3")
 		(at 133.35 64.77 0)
@@
 	)
 	(symbol
-		(lib_id "Switch:SW_DPST_x2")
+		(lib_id "power:GNDREF")
+		(at 167.64 144.78 0)
+		(unit 1)
+		(body_style 1)
+		(exclude_from_sim no)
+		(in_bom yes)
+		(on_board yes)
+		(in_pos_files yes)
+		(dnp no)
+		(fields_autoplaced yes)
+		(property "Reference" "#PWR071"
+			(at 167.64 151.13 0)
+			(hide yes)
+			(show_name no)
+			(do_not_autoplace no)
+			(effects
+				(font
+					(size 1.27 1.27)
+				)
+			)
+		)
+		(property "Value" "GND"
+			(at 167.64 149.86 0)
+			(show_name no)
+			(do_not_autoplace no)
+			(effects
+				(font
+					(size 1.27 1.27)
+				)
+			)
+		)
+		(property "Footprint" ""
+			(at 167.64 144.78 0)
+			(hide yes)
+			(show_name no)
+			(do_not_autoplace no)
+			(effects
+				(font
+					(size 1.27 1.27)
+				)
+			)
+		)
+		(property "Datasheet" ""
+			(at 167.64 144.78 0)
+			(hide yes)
+			(show_name no)
+			(do_not_autoplace no)
+			(effects
+				(font
+					(size 1.27 1.27)
+				)
+			)
+		)
+		(property "Description" "Power symbol creates a global label with name \"GNDREF\" , reference supply ground"
+			(at 167.64 144.78 0)
+			(hide yes)
+			(show_name no)
+			(do_not_autoplace no)
+			(effects
+				(font
+					(size 1.27 1.27)
+				)
+			)
+		)
+		(pin "1"
+		)
+		(instances
+			(project "hardware"
+				(path "/63c7c074-dbc9-4433-b26d-8a099c78afdf/43eeeb2a-883a-4738-8b2b-317d62bf6c96"
+					(reference "#PWR071")
+					(unit 1)
+				)
+			)
+		)
+	)
+	(symbol
+		(lib_id "Connector:Micro_SD_Card_Det1")
+		(at 146.05 130.81 0)
+		(unit 1)
+		(body_style 1)
+		(exclude_from_sim no)
+		(in_bom yes)
+		(on_board yes)
+		(in_pos_files yes)
+		(dnp no)
+		(fields_autoplaced yes)
+		(property "Reference" "J4"
+			(at 146.685 109.22 0)
+			(show_name no)
+			(do_not_autoplace no)
+			(effects
+				(font
+					(size 1.27 1.27)
+				)
+			)
+		)
+		(property "Value" "Micro_SD_Card_Det1"
+			(at 146.685 111.76 0)
+			(show_name no)
+			(do_not_autoplace no)
+			(effects
+				(font
+					(size 1.27 1.27)
+				)
+			)
+		)
+		(property "Footprint" ""
+			(at 198.12 113.03 0)
+			(hide yes)
+			(show_name no)
+			(do_not_autoplace no)
+			(effects
+				(font
+					(size 1.27 1.27)
+				)
+			)
+		)
+		(property "Datasheet" "https://datasheet.lcsc.com/lcsc/2110151630_XKB-Connectivity-XKTF-015-N_C381082.pdf"
+			(at 146.05 128.27 0)
+			(hide yes)
+			(show_name no)
+			(do_not_autoplace no)
+			(effects
+				(font
+					(size 1.27 1.27)
+				)
+			)
+		)
+		(property "Description" "Micro SD Card Socket with one card detection pin"
+			(at 146.05 130.81 0)
+			(hide yes)
+			(show_name no)
+			(do_not_autoplace no)
+			(effects
+				(font
+					(size 1.27 1.27)
+				)
+			)
+		)
+		(pin "4"
+		)
+		(pin "6"
+		)
+		(pin "2"
+		)
+		(pin "7"
+		)
+		(pin "1"
+		)
+		(pin "3"
+		)
+		(pin "5"
+		)
+		(pin "8"
+		)
+		(pin "SH"
+		)
+		(pin "9"
+		)
+		(instances
+			(project "hardware"
+				(path "/63c7c074-dbc9-4433-b26d-8a099c78afdf/43eeeb2a-883a-4738-8b2b-317d62bf6c96"
+					(reference "J4")
+					(unit 1)
+				)
+			)
+		)
+	)
+	(symbol
+		(lib_id "power:PWR_FLAG")
+		(at 102.87 62.23 0)
+		(unit 1)
+		(body_style 1)
+		(exclude_from_sim no)
+		(in_bom yes)
+		(on_board yes)
+		(in_pos_files yes)
+		(dnp no)
+		(fields_autoplaced yes)
+		(property "Reference" "#FLG04"
+			(at 102.87 60.325 0)
+			(hide yes)
+			(show_name no)
+			(do_not_autoplace no)
+			(effects
+				(font
+					(size 1.27 1.27)
+				)
+			)
+		)
+		(property "Value" "PWR_FLAG"
+			(at 102.87 57.15 0)
+			(show_name no)
+			(do_not_autoplace no)
+			(effects
+				(font
+					(size 1.27 1.27)
+				)
+			)
+		)
+		(property "Footprint" ""
+			(at 102.87 62.23 0)
+			(hide yes)
+			(show_name no)
+			(do_not_autoplace no)
+			(effects
+				(font
+					(size 1.27 1.27)
+				)
+			)
+		)
+		(property "Datasheet" ""
+			(at 102.87 62.23 0)
+			(hide yes)
+			(show_name no)
+			(do_not_autoplace no)
+			(effects
+				(font
+					(size 1.27 1.27)
+				)
+			)
+		)
+		(property "Description" "Special symbol for telling ERC where power comes from"
+			(at 102.87 62.23 0)
+			(hide yes)
+			(show_name no)
+			(do_not_autoplace no)
+			(effects
+				(font
+					(size 1.27 1.27)
+				)
+			)
+		)
+		(pin "1"
+		)
+		(instances
+			(project "hardware"
+				(path "/63c7c074-dbc9-4433-b26d-8a099c78afdf/43eeeb2a-883a-4738-8b2b-317d62bf6c96"
+					(reference "#FLG04")
+					(unit 1)
+				)
+			)
+		)
+	)
+	(symbol
+		(lib_id "Switch:SW_SPST")
 		(at 93.98 62.23 0)
 		(unit 1)
@@
 			)
 		)
-		(property "Value" "SW_DPST_x2"
+		(property "Value" "SW_SPST"
 			(at 93.98 58.42 0)
 			(show_name no)
@@
 			)
 		)
-		(property "Description" "Single Pole Single Throw (SPST) switch, separate symbol"
+		(property "Description" "Single Pole Single Throw (SPST) switch"
 			(at 93.98 62.23 0)
 			(hide yes)
@@
 		(pin "1"
 		)
-		(pin "3"
-		)
 		(pin "2"
-		)
-		(pin "4"
 		)
 		(instances
@@
 			)
 		)
-		(property "Footprint" "1079_KEY"
+		(property "Footprint" "footprints:1079_KEY"
 			(at 80.01 62.23 0)
 			(hide yes)
@@
 			)
 		)
-		(property "Value" "01. uF"
+		(property "Value" "0.1 uF"
 			(at 123.19 152.3999 0)
 			(show_name no)
@@
 			)
 		)
-		(property "Value" "680 uF"
+		(property "Value" "180 uF"
 			(at 106.68 73.6599 0)
 			(show_name no)

Commit message: Added capacitor footprints.
Parts:
- C44, C45, C46: footprint (none) -> Capacitor_SMD:C_1206_3216Metric
Changed lines of the file:
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@@
 			)
 		)
-		(property "Footprint" ""
+		(property "Footprint" "Capacitor_SMD:C_1206_3216Metric"
 			(at 194.0052 78.74 0)
 			(hide yes)
@@
 			)
 		)
-		(property "Footprint" ""
+		(property "Footprint" "Capacitor_SMD:C_1206_3216Metric"
 			(at 120.3452 154.94 0)
 			(hide yes)
@@
 			)
 		)
-		(property "Footprint" ""
+		(property "Footprint" "Capacitor_SMD:C_1206_3216Metric"
 			(at 103.8352 76.2 0)
 			(hide yes)

Commit message: Worked on footprints and hardware definations.
Parts:
- C44: footprint Capacitor_SMD:C_1206_3216Metric -> Capacitor_SMD:CP_Elec_8x6.7; Digikey Link (none) -> https://www.digikey.com/en/products/detail/kemet/A768KE187M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; Digikey Part Number (none) -> 399-A768KE187M1ELAE029CT-ND
- C45: footprint Capacitor_SMD:C_1206_3216Metric -> Capacitor_SMD:CP_Elec_10x10; Digikey Link (none) -> https://www.digikey.com/en/products/detail/kemet/A768MS337M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; Digikey Part Number (none) -> 399-A768MS337M1VLAE022CT-ND
- C46: footprint Capacitor_SMD:C_1206_3216Metric -> Capacitor_SMD:C_0805_2012Metric; Digikey Link (none) -> https://www.digikey.com/en/products/detail/kyocera-avx/KGM2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; Digikey Part Number (none) -> 478-KGM21NR71H104KTCT-ND
- J4: footprint (none) -> Connector_Card:microSD_HC_Molex_104031-0811
- L43: footprint (none) -> Inductor_SMD:L_Bourns-SRN8040_8x8.15mm; Digikey Link (none) -> https://www.digikey.com/en/products/detail/bourns-inc/SRN80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; Digikey Part Number (none) -> SRN8040TA-330MCT-ND
- SW41: footprint (none) -> Button_Switch_THT:SW_DIP_SPSTx01_Slide_9.78x4.72mm_W7.62mm_P2.54mm
Changed lines of the file:
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@@
 			)
 		)
-		(property "Footprint" "Capacitor_SMD:C_1206_3216Metric"
+		(property "Footprint" "Capacitor_SMD:CP_Elec_10x10"
 			(at 194.0052 78.74 0)
 			(hide yes)
@@
 		)
 		(property "Description" "Unpolarized capacitor"
+			(at 193.04 74.93 0)
+			(hide yes)
+			(show_name no)
+			(do_not_autoplace no)
+			(effects
+				(font
+					(size 1.27 1.27)
+				)
+			)
+		)
+		(property "Digikey Link" "https://www.digikey.com/en/products/detail/kemet/A768MS337M1VLAE022/12705376"
+			(at 193.04 74.93 0)
+			(hide yes)
+			(show_name no)
+			(do_not_autoplace no)
+			(effects
+				(font
+					(size 1.27 1.27)
+				)
+			)
+		)
+		(property "Digikey Part Number" "399-A768MS337M1VLAE022CT-ND"
 			(at 193.04 74.93 0)
 			(hide yes)
@@
 			)
 		)
-		(property "Footprint" ""
+		(property "Footprint" "Connector_Card:microSD_HC_Molex_104031-0811"
 			(at 198.12 113.03 0)
 			(hide yes)
@@
 			)
 		)
-		(property "Footprint" ""
+		(property "Footprint" "Button_Switch_THT:SW_DIP_SPSTx01_Slide_9.78x4.72mm_W7.62mm_P2.54mm"
 			(at 93.98 62.23 0)
 			(hide yes)
@@
 			)
 		)
-		(property "Footprint" ""
+		(property "Footprint" "Inductor_SMD:L_Bourns-SRN8040_8x8.15mm"
 			(at 171.45 67.31 0)
 			(hide yes)
@@
 		(property "Description" "Inductor"
 			(at 171.45 67.31 0)
+			(hide yes)
+			(show_name no)
+			(do_not_autoplace no)
+			(effects
+				(font
+					(size 1.27 1.27)
+				)
+			)
+		)
+		(property "Digikey Link" "https://www.digikey.com/en/products/detail/bourns-inc/SRN8040TA-330M/6155132"
+			(at 171.45 67.31 90)
+			(hide yes)
+			(show_name no)
+			(do_not_autoplace no)
+			(effects
+				(font
+					(size 1.27 1.27)
+				)
+			)
+		)
+		(property "Digikey Part Number" "SRN8040TA-330MCT-ND"
+			(at 171.45 67.31 90)
 			(hide yes)
 			(show_name no)
@@
 			)
 		)
-		(property "Footprint" "Capacitor_SMD:C_1206_3216Metric"
+		(property "Footprint" "Capacitor_SMD:C_0805_2012Metric"
 			(at 120.3452 154.94 0)
 			(hide yes)
@@
 		)
 		(property "Description" "Unpolarized capacitor"
+			(at 119.38 151.13 0)
+			(hide yes)
+			(show_name no)
+			(do_not_autoplace no)
+			(effects
+				(font
+					(size 1.27 1.27)
+				)
+			)
+		)
+		(property "Digikey Link" "https://www.digikey.com/en/products/detail/kyocera-avx/KGM21NR71H104KT/563505"
+			(at 119.38 151.13 0)
+			(hide yes)
+			(show_name no)
+			(do_not_autoplace no)
+			(effects
+				(font
+					(size 1.27 1.27)
+				)
+			)
+		)
+		(property "Digikey Part Number" "478-KGM21NR71H104KTCT-ND"
 			(at 119.38 151.13 0)
 			(hide yes)
@@
 			)
 		)
-		(property "Footprint" "Capacitor_SMD:C_1206_3216Metric"
+		(property "Footprint" "Capacitor_SMD:CP_Elec_8x6.7"
 			(at 103.8352 76.2 0)
 			(hide yes)
@@
 			(at 102.87 72.39 0)
 			(hide yes)
+			(show_name no)
+			(do_not_autoplace no)
+			(effects
+				(font
+					(size 1.27 1.27)
+				)
+			)
+		)
+		(property "Digikey Link" "https://www.digikey.com/en/products/detail/kemet/A768KE187M1ELAE029/13420143"
+			(at 102.87 72.39 0)
+			(hide yes)
+			(show_name no)
+			(do_not_autoplace no)
+			(effects
+				(font
+					(size 1.27 1.27)
+				)
+			)
+		)
+		(property "Digikey Part Number" "399-A768KE187M1ELAE029CT-ND"
+			(at 102.87 72.39 0)
+			(hide yes)

Commit message: Worked on PCB routing and component placement.
Parts:
- B41: Digikey Link (none) -> https://www.digikey.com/en/products/detail/keystone-electro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; Digikey Part Number (none) -> 36-1079-ND
- D41: footprint Diode_THT:D_DO-201AD_P15.24mm_Horizontal -> Diode_THT:D_A-405_P7.62mm_Horizontal; Digikey Link (none) -> https://www.digikey.com/en/products/detail/diotec-semicondu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; Digikey Part Number (none) -> 4878-1N5820CT-ND
- J4: Digikey Link (none) -> https://www.digikey.com/en/products/detail/molex/1040310811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; Digikey Part Number (none) -> WM6357CT-ND
- U8: Digikey Link (none) -> https://www.digikey.com/en/products/detail/umw/LM2596S-3-3/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; Digikey Part Number (none) -> 4518-LM2596S-3.3CT-ND
Changed lines of the file:
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@@
+			)
+		)
+		(property "Digikey Link" "https://www.digikey.com/en/products/detail/umw/LM2596S-3-3/16705894"
+			(at 133.35 64.77 0)
+			(hide yes)
+			(show_name no)
+			(do_not_autoplace no)
+			(effects
+				(font
+					(size 1.27 1.27)
+				)
+			)
+		)
+		(property "Digikey Part Number" "4518-LM2596S-3.3CT-ND"
+			(at 133.35 64.77 0)
+			(hide yes)
+			(show_name no)
+			(do_not_autoplace no)
+			(effects
+				(font
+					(size 1.27 1.27)
+				)
 			)
 		)
@@
 			)
 		)
-		(property "Footprint" "Diode_THT:D_DO-201AD_P15.24mm_Horizontal"
+		(property "Footprint" "Diode_THT:D_A-405_P7.62mm_Horizontal"
 			(at 150.495 74.93 0)
 			(hide yes)
@@
 			)
 		)
+		(property "Digikey Link" "https://www.digikey.com/en/products/detail/diotec-semiconductor/1N5820/22191764"
+			(at 154.94 74.93 90)
+			(hide yes)
+			(show_name no)
+			(do_not_autoplace no)
+			(effects
+				(font
+					(size 1.27 1.27)
+				)
+			)
+		)
+		(property "Digikey Part Number" "4878-1N5820CT-ND"
+			(at 154.94 74.93 90)
+			(hide yes)
+			(show_name no)
+			(do_not_autoplace no)
+			(effects
+				(font
+					(size 1.27 1.27)
+				)
+			)
+		)
 		(pin "2"
 		)
@@
 			)
 		)
+		(property "Digikey Link" "https://www.digikey.com/en/products/detail/molex/1040310811/2370379"
+			(at 146.05 130.81 0)
+			(hide yes)
+			(show_name no)
+			(do_not_autoplace no)
+			(effects
+				(font
+					(size 1.27 1.27)
+				)
+			)
+		)
+		(property "Digikey Part Number" "WM6357CT-ND"
+			(at 146.05 130.81 0)
+			(hide yes)
+			(show_name no)
+			(do_not_autoplace no)
+			(effects
+				(font
+					(size 1.27 1.27)
+				)
+			)
+		)
 		(pin "4"
 		)
@@
 			(at 80.01 62.23 0)
 			(hide yes)
+			(show_name no)
+			(do_not_autoplace no)
+			(effects
+				(font
+					(size 1.27 1.27)
+				)
+			)
+		)
+		(property "Digikey Link" "https://www.digikey.com/en/products/detail/keystone-electronics/1079/5118843"
+			(at 80.01 62.23 0)
+			(hide yes)
+			(show_name no)
+			(do_not_autoplace no)
+			(effects
+				(font
+					(size 1.27 1.27)
+				)
+			)
+		)
+		(property "Digikey Part Number" "36-1079-ND"
+			(at 80.01 62.23 0)
+			(hide yes)
