File: hardware/hardware.kicad_pcb (KiCad board)
At the start: 4 copper layers, 220 x 108 mm, 88 parts, among them J1 SMA, J2 Test Header, J4 Micro_SD_Card_Det1, P5 BMIS-202-C, SW41 SW_SPST, U1 CC1101, U2 CC1190, U3 B39921B3588U410, U4 ADS1115IDGS, U5 BME280, U6 MS5611-01BA, U7 NEO-M9N, U8 LM2596S-3.3, X1 26.000 MHz

Commit message: Fixed I2C1 global labels.
Connections:
- A1 pad 31: I2C0_SCL -> I2C1_SCL
- A1 pad 32: I2C0_SDA -> I2C1_SDA
- R12 pad 1: I2C0_SDA -> I2C1_SDA
- R13 pad 1: I2C0_SCL -> I2C1_SCL
- U6 pad 7: I2C0_SDA -> I2C1_SDA
- U6 pad 8: I2C0_SCL -> I2C1_SCL
Changed lines of the file:
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@@
 		(capping no)
 		(filling no)
-		(zone_defaults)
 		(pcbplotparams
 			(layerselection 0x00000000_00000000_55555555_5755f5ff)
@@
 			(unit
 				(name "A")
-				(pins "5" "6" "20" "21" "18" "19" "4" "1" "8" "2" "23" "22" "7" "10"
-					"12" "13" "24" "9" "15" "16" "17" "14" "11" "3"
+				(pins "5" "6" "20" "21" "18" "19" "4" "1" "8" "2" "23" "22" "7" "24"
+					"13" "12" "10" "9" "15" "16" "17" "14" "11" "3"
 				)
 			)
@@
 			(layers "F.Cu" "F.Mask" "F.Paste")
 			(roundrect_rratio 0.222222)
-			(net "I2C0_SCL")
+			(net "I2C1_SCL")
 			(pintype "passive")
 		)
@@
 			(size 0.95 0.55)
 			(layers "F.Cu" "F.Mask" "F.Paste")
-			(net "I2C0_SDA")
+			(net "I2C1_SDA")
 			(pinfunction "SDI/SDA_7")
 			(pintype "bidirectional")
@@
 			(size 0.95 0.55)
 			(layers "F.Cu" "F.Mask" "F.Paste")
-			(net "I2C0_SCL")
+			(net "I2C1_SCL")
 			(pinfunction "SCLK_8")
 			(pintype "input")
@@
 				(name "A")
 				(pins "30" "37" "1" "2" "4" "5" "6" "7" "9" "10" "11" "12" "14" "15"
-					"16" "17" "19" "20" "39" "40" "3" "23" "28" "18" "13" "38" "8" "36"
+					"16" "17" "19" "20" "39" "40" "23" "3" "8" "38" "13" "28" "18" "36"
 					"21" "22" "24" "25" "26" "27" "29" "35" "31" "32" "34" "33"
 				)
@@
 			(layers "F.Cu" "F.Mask")
 			(roundrect_rratio 0.5)
-			(net "I2C0_SCL")
+			(net "I2C1_SCL")
 			(pinfunction "GPIO26_ADC0_31")
 			(pintype "bidirectional")
@@
 			(layers "F.Cu" "F.Mask")
 			(roundrect_rratio 0.5)
-			(net "I2C0_SDA")
+			(net "I2C1_SDA")
 			(pinfunction "GPIO27_ADC1_32")
 			(pintype "bidirectional")
@@
 			(layers "F.Cu" "F.Mask" "F.Paste")
 			(roundrect_rratio 0.222222)
-			(net "I2C0_SDA")
+			(net "I2C1_SDA")
 			(pintype "passive")
 		)

Commit message: Worked on PCB routing and component placement.
Parts:
- added R3: 10K, Resistor_SMD:R_0603_1608Metric, F.Cu at (55.6, 111.0)
- added R4: 10K, Resistor_SMD:R_0603_1608Metric, F.Cu at (58.1, 111.0)
- added R5: 10K, Resistor_SMD:R_0603_1608Metric, F.Cu at (60.7, 111.0)
- C44, C45, C46, L43, SW41, U8: moved to B.Cu
- D41: footprint Diode_THT:D_DO-201AD_P15.24mm_Horizontal -> Diode_THT:D_A-405_P7.62mm_Horizontal; moved to B.Cu
- P5: value BMIS-202-C -> BMI-S-205-C; footprint RF_Shielding:Laird_Technologies_BMI-S-202-F_16.50x16.50mm -> RF_Shielding:Laird_Technologies_BMI-S-203-F_26.21x26.21mm
- R04, R07, R08, R1, R11, R12, R13, R14, R141, R15, R151, R16, R161, R171, R2: footprint Resistor_SMD:R_1206_3216Metric -> Resistor_SMD:R_0603_1608Metric
- X1: footprint Crystal:Crystal_SMD_3225-4Pin_3.2x2.5mm -> Crystal:Crystal_SMD_2016-4Pin_2.0x1.6mm
- moved C02 138.2 mm to (244.5, 58.2)
- moved D2 134.6 mm to (65.0, 55.0), turned to -90 degrees
- moved D1 134.4 mm to (56.0, 55.3), turned to -90 degrees
- moved R1 121.7 mm to (56.0, 64.3), turned to 90 degrees
- moved R2 121.5 mm to (65.0, 64.3), turned to 90 degrees
- moved SW41 100.2 mm to (113.7, 60.7), turned to 180 degrees
- moved J4 99.7 mm to (43.0, 60.2), turned to 180 degrees
- moved R151 97.0 mm to (57.4, 89.5), turned to -90 degrees
- moved C44 95.2 mm to (110.2, 70.4), turned to 180 degrees
- moved R161 94.0 mm to (55.9, 89.5), turned to -90 degrees
- moved C161 93.7 mm to (56.4, 86.7), turned to 180 degrees
- moved C45 93.6 mm to (108.0, 82.7), turned to 180 degrees
- moved R16 89.9 mm to (155.2, 69.3), turned to 180 degrees
- moved C181 87.9 mm to (88.1, 113.7), turned to -90 degrees
- moved C132 87.5 mm to (61.1, 90.4)
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Connections:
- U2 pad 6: HGM -> Net-(U2-HGM)
- U2 pad 7: LNA_EN -> Net-(U2-LNA_EN)
- U2 pad 8: PA_EN -> Net-(U2-PA_EN)
Routing:
- net GND: track 4.41 -> 47.1 mm
- net Net-(C161-Pad1): track 0.00 -> 33.7 mm
- net VDD: track 0.00 -> 15.4 mm, vias 0 -> 2
- net Net-(J1-In): track 0.00 -> 12.5 mm
- net Net-(C25-Pad1): track 0.00 -> 4.35 mm
- net Net-(U2-VDD_PA1): track 0.00 -> 3.36 mm
- net Net-(U2-VDD_LNA): track 0.00 -> 3.35 mm
- net Net-(U2-VDD_PA2): track 0.00 -> 2.84 mm
- net Net-(U2-BIAS): track 0.00 -> 1.95 mm
- net Net-(U2-PA_OUT): track 0.00 -> 1.42 mm
Other:
- board size 220 x 108 mm -> 220 x 111.8 mm

Commit message: Worked more on the PCB layout.
Parts:
- moved TP1 22.8 mm to (101.0, 100.0)
- moved TP2 22.8 mm to (101.0, 95.4)
- moved R07 2.56 mm to (148.0, 82.7), turned to -90 degrees
- moved R08 2.56 mm to (145.4, 82.7), turned to -90 degrees
- moved C52 1.28 mm to (59.7, 98.0)
- moved C41 0.72 mm to (91.1, 108.5)
- moved C51 0.72 mm to (91.1, 106.5)
- moved C101 0.57 mm to (84.2, 96.2), turned to 0 degrees
- turned C1 to 0 degrees
- turned C121 to -90 degrees
- turned L121 to 0 degrees
- turned L122 to -90 degrees
- turned L131 to 0 degrees
- turned L132 to 0 degrees
- turned L43 to 0 degrees
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Routing:
- net GND: track 47.1 -> 195.1 mm, vias 0 -> 22
- net VDD: track 15.4 -> 100.7 mm, vias 2 -> 8
- net SPI1_TX: track 0.00 -> 54.0 mm
- net SPI1_RX: track 0.00 -> 44.3 mm
- net SPI1_CSn: track 0.00 -> 42.4 mm
- net Net-(U1-XOSC_Q1): track 0.00 -> 42.2 mm
- net Net-(U1-DGUARD): track 0.00 -> 41.3 mm
- net Net-(D41-K): track 0.00 -> 27.3 mm
- net Net-(SW41-B): track 0.00 -> 25.1 mm
- net Net-(U1-GDO2): track 0.00 -> 24.2 mm
- net Net-(U2-HGM): track 0.00 -> 19.1 mm
- net Net-(U2-PA_EN): track 0.00 -> 19.0 mm
- net Net-(U1-XOSC_Q2): track 0.00 -> 18.9 mm
- net Net-(U2-LNA_EN): track 0.00 -> 18.4 mm
- net Net-(B41-Pad2): track 0.00 -> 18.3 mm
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